File: PCB/KiCad/ESP32AY.kicad_pcb (KiCad board)
At the start: 2 copper layers, 55 x 100 mm, 112 parts, among them J1 USB_C_Receptacle_USB2.0_14P, J2 MiniJack, J3 SD Card, Q1 BC807, Q2 BC817, Q3 BC817, SW1 Check bat, SW2 EN, SW3 BOOT, U1 AY-3-8910, U2 AY-3-8910, U3 CH340G, U4 ESP32-WROOM-32, U5 TPA6130A2RTJTG4, U6 IP5306, U7 AMS1117-3.3, U8 74HC595, U9 74HC595, Y3 12MHz

Commit message: initial C3 schematic, pcb, code.
Parts:
- removed the C21 at (36.3, 111.2)
- removed the R24 at (34.0, 102.4)
- removed the R25 at (25.9, 99.0)
- removed the R36 at (50.0, 110.9)
- removed the R37 at (44.8, 93.2)
- removed the R38 at (54.1, 111.9)
- removed the R39 at (66.2, 94.6)
- removed the R40 at (31.7, 94.8)
- removed the SW1 at (22.1, 99.3)
- removed the U4 at (50.0, 35.9)
- removed the U6 at (28.1, 103.0)
- added C14: 22uf, Capacitor_SMD:C_1206_3216Metric_Pad1.33x1.80mm_HandSolder, B.Cu at (26.7, 96.1)
- added C15: 100n, Capacitor_SMD:C_0805_2012Metric_Pad1.18x1.45mm_HandSolder, B.Cu at (22.2, 37.5)
- added C16: 22uf, Capacitor_SMD:C_1206_3216Metric_Pad1.33x1.80mm_HandSolder, B.Cu at (32.2, 94.7)
- added C17: 100n, Capacitor_SMD:C_0805_2012Metric_Pad1.18x1.45mm_HandSolder, B.Cu at (35.9, 34.4)
- added C24: 10uf, Capacitor_SMD:C_0805_2012Metric_Pad1.18x1.45mm_HandSolder, F.Cu at (33.7, 27.8)
- added C25: 100n, Capacitor_SMD:C_0805_2012Metric_Pad1.18x1.45mm_HandSolder, F.Cu at (29.3, 27.8)
- added C26: 10uf, Capacitor_SMD:C_0805_2012Metric_Pad1.18x1.45mm_HandSolder, B.Cu at (31.2, 56.0)
- added C27: 2.2nf, Capacitor_SMD:C_0805_2012Metric_Pad1.18x1.45mm_HandSolder, B.Cu at (27.4, 56.0)
- added C28: 10uf, Capacitor_SMD:C_0805_2012Metric_Pad1.18x1.45mm_HandSolder, B.Cu at (31.2, 61.8)
- added C29: 10uf, Capacitor_SMD:C_0805_2012Metric_Pad1.18x1.45mm_HandSolder, B.Cu at (34.8, 47.2)
- added C31: 100n, Capacitor_SMD:C_0805_2012Metric_Pad1.18x1.45mm_HandSolder, B.Cu at (34.8, 44.9)
- added D4: SS14, Diode_SMD:D_SMA, B.Cu at (30.5, 99.5)
- added J2: Battery, Connector_JST:JST_PH_S2B-PH-K_1x02_P2.00mm_Horizontal, B.Cu at (40.5, 91.0)
- added Q1: IRLML6402, Package_TO_SOT_SMD:SOT-23, F.Cu at (31.9, 94.3)
- added R15: 47k, Resistor_SMD:R_0805_2012Metric_Pad1.20x1.40mm_HandSolder, F.Cu at (27.4, 98.8)
- added R16: 6.2k, Resistor_SMD:R_0805_2012Metric_Pad1.20x1.40mm_HandSolder, F.Cu at (27.4, 102.8)
- added R17: 1k, Resistor_SMD:R_0805_2012Metric_Pad1.20x1.40mm_HandSolder, F.Cu at (21.9, 103.1)
- added R22: 10K, Resistor_SMD:R_0805_2012Metric_Pad1.20x1.40mm_HandSolder, B.Cu at (22.1, 45.2)
- added R23: 10K, Resistor_SMD:R_0805_2012Metric_Pad1.20x1.40mm_HandSolder, B.Cu at (22.1, 43.2)
- added R4: 1k, Resistor_SMD:R_0805_2012Metric_Pad1.20x1.40mm_HandSolder, F.Cu at (26.6, 109.7)
- added R44: 1K, Resistor_SMD:R_0805_2012Metric_Pad1.20x1.40mm_HandSolder, B.Cu at (32.4, 65.1)
- added R45: 1K, Resistor_SMD:R_0805_2012Metric_Pad1.20x1.40mm_HandSolder, B.Cu at (32.1, 58.9)
- added R8: 2k*, Resistor_SMD:R_0805_2012Metric_Pad1.20x1.40mm_HandSolder, B.Cu at (40.6, 110.1)
- added R9: 10K, Resistor_SMD:R_0805_2012Metric_Pad1.20x1.40mm_HandSolder, F.Cu at (27.7, 94.4)
- added U1: PCF8574AT, Package_SO:SOIC-16W_7.5x10.3mm_P1.27mm, F.Cu at (48.6, 114.6)
- added U10: MB85RC256V, Package_SO:SOIC-8_3.9x4.9mm_P1.27mm, B.Cu at (28.5, 31.5)
- added U11: PCM5102A, Package_SO:TSSOP-20_4.4x6.5mm_P0.65mm, B.Cu at (28.8, 43.5)
- added U12: ESP32-WROVER-E, mod:ESP32-WROVER-IE, B.Cu at (50.0, 35.7)
- added U5: TP4056, Package_SO:SOIC-8-1EP_3.9x4.9mm_P1.27mm_EP2.41x3.3mm_ThermalVias, B.Cu at (35.0, 103.5)
- added U8: SDB628, Package_TO_SOT_SMD:SOT-23-6_Handsoldering, B.Cu at (25.9, 101.1)
- added U9: DS3231MZ, Package_SO:SOIC-8_3.9x4.9mm_P1.27mm, B.Cu at (28.5, 37.1)
- BAT+1: value BAT+ -> +
- BAT-1: value BAT- -> -
- C10: renamed from C19; footprint Capacitor_SMD:C_0805_2012Metric_Pad1.18x1.45mm_HandSolder -> Capacitor_SMD:C_1206_3216Metric_Pad1.33x1.80mm_HandSolder
- C11: renamed from C32; moved to B.Cu
- C19: renamed from C31; moved to B.Cu
- C21: renamed from C27; moved to B.Cu
- C22: value 22uf -> 100n
- C23: value 22uf -> 2.2uf; footprint Capacitor_SMD:C_0805_2012Metric -> Capacitor_SMD:C_0805_2012Metric_Pad1.18x1.45mm_HandSolder
- C30: value 22uf -> 2.2nf
- C6: renamed from C17; moved to B.Cu
- C9: renamed from C20; moved to B.Cu
- D1: value 25% -> OK
- D2: value 50% -> CHRG
- D3: value 75% -> PMEG4010CEJ; footprint LED_SMD:LED_0805_2012Metric -> Diode_SMD:D_SOD-323F
- D5: renamed from D4; value 100% -> PWR
- L1: value 1UH -> 22uH; footprint Inductor_SMD:L_7.3x7.3_H3.5 -> Inductor_SMD:L_Bourns_SRN8040TA
- R10: renamed from R6; value 100K -> 1M
- R11: renamed from R7; value 10K -> 100K
- R12: renamed from R35; moved to B.Cu
- R13: renamed from R31; moved to F.Cu
- R24: renamed from R1; moved to B.Cu
- R3: renamed from R23; footprint Resistor_SMD:R_0805_2012Metric -> Resistor_SMD:R_0805_2012Metric_Pad1.20x1.40mm_HandSolder; moved to B.Cu
- R40: renamed from R26; moved to F.Cu
- R41: renamed from R27; moved to F.Cu
- R5: renamed from R19; moved to B.Cu
- R6: renamed from R18; moved to B.Cu
- R7: renamed from R34; moved to B.Cu
- U13: renamed from U3; value CH340G -> CH340C
- U3: renamed from U8; footprint Package_SO:SO-16_5.3x10.2mm_P1.27mm -> Package_SO:SO-16_3.9x9.9mm_P1.27mm
- U4: renamed from U9; footprint Package_SO:SO-16_5.3x10.2mm_P1.27mm -> Package_SO:SO-16_3.9x9.9mm_P1.27mm
- moved C22 72.1 mm to (22.1, 39.7), turned to 180 degrees
- moved R26 66.3 mm to (72.3, 91.6), turned to 90 degrees
- moved R27 63.3 mm to (70.3, 91.6), turned to 90 degrees
- moved C23 61.0 mm to (22.1, 47.2), turned to 180 degrees
- moved R6 37.1 mm to (52.8, 116.9), turned to 0 degrees
- moved C30 36.8 mm to (27.3, 61.8), turned to 180 degrees
- moved R5 36.2 mm to (52.8, 118.9), turned to 180 degrees
- moved C9 29.1 mm to (49.0, 115.9), turned to -90 degrees
- moved L1 24.7 mm to (26.1, 107.4), turned to 0 degrees
- moved R7 24.7 mm to (51.7, 113.9), turned to 90 degrees
- moved D3 18.0 mm to (36.6, 93.2), turned to 90 degrees
- moved C6 14.8 mm to (38.4, 110.1), turned to 90 degrees
- moved C21 12.0 mm to (62.1, 28.7), turned to 90 degrees
- moved R3 11.3 mm to (36.2, 110.1), turned to 90 degrees
- moved R10 11.1 mm to (59.3, 29.1), turned to 0 degrees
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- renumbered C4 to C1, C2 to C12, C28 to C13, C1 to C18, C3 to C2, C29 to C20, C16 to C3, C11 to C32, C12 to C33, C13 to C34, C14 to C35, C33 to C36, C34 to C37, C10 to C38, C5 to C39, C26 to C4, C15 to C40, C9 to C41, C8 to C42, C7 to C43, C6 to C44, C24 to C5, C25 to C7, C18 to C8, J2 to J4, Q1 to Q2, Q2 to Q3, Q3 to Q4, R41 to R1, R29 to R14, R20 to R18, R3 to R19, R42 to R2, R28 to R20, R30 to R21, R2 to R25, R21 to R26, R22 to R27, R4 to R28, R5 to R29, R12 to R30, R9 to R31, R17 to R32, R14 to R33, R33 to R34, R32 to R35, R11 to R36, R10 to R37, R16 to R38, R15 to R39, R13 to R42, R8 to R43, S2 to S1, S4 to S2, S6 to S3, SW3 to SW1, U5 to U14, U7 to U2, U1 to U6, U2 to U7, Y3 to Y1
Connections:
- net BT_DN renamed BTN_DN
- net BT_UP renamed BTN_UP
- C22 pad 1: Net-(U6-Vout) -> +3.3V
- C23 pad 1: Net-(U6-Vout) -> Net-(U11-CAPM)
- C23 pad 2: GND -> Net-(U11-CAPP)
- C30 pad 1: GND -> PCM_R
- C30 pad 2: Net-(U6-BAT) -> GND
- D2 pad 1: Net-(D1-A) -> Net-(D2-K)
- D2 pad 2: Net-(D1-K) -> Net-(D1-A)
- D3 pad 1: Net-(D1-K) -> STPUP_VIN
- D3 pad 2: Net-(D3-A) -> Vin
- D5 pad 1: Net-(D3-A) -> GND
- D5 pad 2: Net-(D1-K) -> Net-(D5-A)
- Encoder1 pad MP: (no net) -> GND
- L1 pad 1: Net-(U6-SW) -> Net-(U8-EN)
- L1 pad 2: Bat+ -> Net-(D4-A)
- R34 pad 2: DAC_SOUND_R -> DAC_DAT
- R35 pad 2: DAC_SOUND_L -> DAC_BCK
- S3 pad 1: Net-(U6-Vout) -> Net-(U8-EN)
- S3 pad 2: Net-(U6-Vout) -> STPUP_VIN
- S3 pad 3: +5V -> STPUP_VIN
Routing:
- net GND: track 122.1 -> 852.0 mm, vias 98 -> 66
- net +3.3V: track 291.9 -> 422.0 mm, vias 13 -> 26
- net ENC_B: track 118.4 -> 6.87 mm, vias 3 -> 1
- net BTN_DN: track 120.1 -> 32.2 mm, vias 3 -> 0
- net DAC_DAT: track 0.00 -> 87.8 mm, vias 0 -> 6
- net USB_SENS: track 94.1 -> 6.60 mm, vias 5 -> 1
- net Net-(U12-IO1/TXD0): track 2.83 -> 82.7 mm
- net Net-(U12-IO3/RXD0): track 2.89 -> 81.6 mm
- net Bat+: track 90.5 -> 169.2 mm, vias 9 -> 6
- net DAC_BCK: track 0.00 -> 78.4 mm, vias 0 -> 6
- net ENC_OK: track 96.4 -> 18.1 mm, vias 1 -> 0
- net TX0: track 87.1 -> 10.3 mm
- net RX0: track 83.2 -> 7.21 mm
- net DAC_SOUND_L: track 74.6 -> 0.00 mm, vias 6 -> 0
- net ENC_A: track 85.8 -> 12.2 mm, vias 7 -> 1
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Other:
- board text added: "+"
- board text added: "Battery"
- board text added: "ZxPod player Rev.C3 by Spawn Andy Karpov 2025"
- board text removed: "ZxPod player Rev. C by Spawn 2025"
