File: PCB/KiCad/ESP32AY.kicad_sch (KiCad schematic)
At the start: 107 parts, among them J1 USB_C_Receptacle_USB2.0_14P, J2 MiniJack, J3 SD Card, Q1 BC807, Q2 BC817, Q3 BC817, SW1 Check bat, SW2 EN, SW3 BOOT, U1 AY-3-8910, U2 AY-3-8910, U3 CH340G, U4 ESP32-WROOM-32, U5 TPA6130A2RTJTG4, U6 IP5306, U7 AMS1117-3.3, U8 74HC595, U9 74HC595, Y3 12MHz

Commit message: initial C3 schematic, pcb, code.
Parts:
- removed C21: 22uf, Capacitor_SMD:C_0805_2012Metric_Pad1.18x1.45mm_HandSolder, symbol Device:C_Small
- removed D3: 75%, LED_SMD:LED_0805_2012Metric, symbol Device:LED
- removed R24: 0.5R, Resistor_SMD:R_0805_2012Metric, symbol Device:R_Small
- removed R25: 10K, Resistor_SMD:R_0805_2012Metric, symbol Device:R_Small
- removed R36, R37, R38, R39, R40: 10K, Resistor_SMD:R_0805_2012Metric_Pad1.20x1.40mm_HandSolder, symbol Device:R_Small
- removed SW1: Check bat, Jumper:SolderJumper-2_P1.3mm_Open_RoundedPad1.0x1.5mm, symbol Switch:SW_Push
- removed U4: ESP32-WROOM-32, RF_Module:ESP32-WROOM-32, symbol RF_Module:ESP32-WROOM-32
- removed U6: IP5306, Package_SO:HSOP-8-1EP_3.9x4.9mm_P1.27mm_EP2.41x3.1mm, symbol Module:SM5308
- added C14, C16: 22uf, Capacitor_SMD:C_1206_3216Metric_Pad1.33x1.80mm_HandSolder, symbol Device:C_Small
- added C15, C17, C25, C31: 100n, Capacitor_SMD:C_0805_2012Metric_Pad1.18x1.45mm_HandSolder, symbol Device:C_Small
- added C24, C26, C28, C29: 10uf, Capacitor_SMD:C_0805_2012Metric_Pad1.18x1.45mm_HandSolder, symbol Device:C_Small
- added C27: 2.2nf, Capacitor_SMD:C_0805_2012Metric_Pad1.18x1.45mm_HandSolder, symbol Device:C_Small
- added D3: PMEG4010CEJ, Diode_SMD:D_SOD-323F, symbol Diode:PMEG4010CEJ
- added D4: SS14, Diode_SMD:D_SMA, symbol Diode:SS14
- added J2: Battery, Connector_JST:JST_PH_S2B-PH-K_1x02_P2.00mm_Horizontal, symbol SparkFun-Connectors:CONN_02-JST-2MM-SMT
- added Q1: IRLML6402, Package_TO_SOT_SMD:SOT-23, symbol Transistor_FET:IRLML6402
- added R15: 47k, Resistor_SMD:R_0805_2012Metric_Pad1.20x1.40mm_HandSolder, symbol Device:R_Small
- added R16: 6.2k, Resistor_SMD:R_0805_2012Metric_Pad1.20x1.40mm_HandSolder, symbol Device:R_Small
- added R17, R4: 1k, Resistor_SMD:R_0805_2012Metric_Pad1.20x1.40mm_HandSolder, symbol Device:R_Small
- added R22, R23, R9: 10K, Resistor_SMD:R_0805_2012Metric_Pad1.20x1.40mm_HandSolder, symbol Device:R_Small
- added R44, R45: 1K, Resistor_SMD:R_0805_2012Metric_Pad1.20x1.40mm_HandSolder, symbol Device:R_Small
- added R8: 2k*, Resistor_SMD:R_0805_2012Metric_Pad1.20x1.40mm_HandSolder, symbol Device:R_Small
- added U1: PCF8574AT, Package_SO:SOIC-16W_7.5x10.3mm_P1.27mm, symbol Interface_Expansion:PCF8574AT
- added U10: MB85RC256V, Package_SO:SOIC-8_3.9x4.9mm_P1.27mm, symbol Memory_EEPROM:24LC256
- added U11: PCM5102A, Package_SO:TSSOP-20_4.4x6.5mm_P0.65mm, symbol Audio:PCM5102A
- added U12: ESP32-WROVER-E, mod:ESP32-WROVER-IE, symbol ESP32-WROVER:ESP32-WROVER-E
- added U5: TP4056, Package_SO:SOIC-8-1EP_3.9x4.9mm_P1.27mm_EP2.41x3.3mm_ThermalVias, symbol Battery_Management:TP4056-42-ESOP8
- added U8: SDB628, Package_TO_SOT_SMD:SOT-23-6_Handsoldering, symbol retro:SDB628
- added U9: DS3231MZ, Package_SO:SOIC-8_3.9x4.9mm_P1.27mm, symbol Timer_RTC:DS3231MZ
- BAT+1: value BAT+ -> +
- BAT-1: value BAT- -> -
- C10: renamed from C19; footprint Capacitor_SMD:C_0805_2012Metric_Pad1.18x1.45mm_HandSolder -> Capacitor_SMD:C_1206_3216Metric_Pad1.33x1.80mm_HandSolder
- C22: value 22uf -> 100n
- C23: value 22uf -> 2.2uf; footprint Capacitor_SMD:C_0805_2012Metric -> Capacitor_SMD:C_0805_2012Metric_Pad1.18x1.45mm_HandSolder
- C30: value 22uf -> 2.2nf
- C36: renamed from C33; now not fitted; now left out of the parts list
- C37: renamed from C34; now not fitted; now left out of the parts list
- D1: value 25% -> OK
- D2: value 50% -> CHRG
- D5: renamed from D4; value 100% -> PWR
- L1: value 1UH -> 22uH; footprint Inductor_SMD:L_7.3x7.3_H3.5 -> Inductor_SMD:L_Bourns_SRN8040TA
- R10: renamed from R6; value 100K -> 1M
- R11: renamed from R7; value 10K -> 100K
- R3: renamed from R23; footprint Resistor_SMD:R_0805_2012Metric -> Resistor_SMD:R_0805_2012Metric_Pad1.20x1.40mm_HandSolder
- R34: renamed from R33; now not fitted; now left out of the parts list
- R35: renamed from R32; now not fitted; now left out of the parts list
- U13: renamed from U3; value CH340G -> CH340C
- U3: renamed from U8; footprint Package_SO:SO-16_5.3x10.2mm_P1.27mm -> Package_SO:SO-16_3.9x9.9mm_P1.27mm
- U4: renamed from U9; footprint Package_SO:SO-16_5.3x10.2mm_P1.27mm -> Package_SO:SO-16_3.9x9.9mm_P1.27mm
- Y1: renamed from Y3; now not fitted; now left out of the parts list
- renumbered C4 to C1, C32 to C11, C2 to C12, C28 to C13, C1 to C18, C31 to C19, C3 to C2, C29 to C20, C27 to C21, C16 to C3, C11 to C32, C12 to C33, C13 to C34, C14 to C35, C10 to C38, C5 to C39, C26 to C4, C15 to C40, C9 to C41, C8 to C42, C7 to C43, C6 to C44, C24 to C5, C17 to C6, C25 to C7, C18 to C8, C20 to C9, J2 to J4, Q1 to Q2, Q2 to Q3, Q3 to Q4, R41 to R1, R35 to R12, R31 to R13, R29 to R14, R20 to R18, R3 to R19, R42 to R2, R28 to R20, R30 to R21, R1 to R24, R2 to R25, R21 to R26, R22 to R27, R4 to R28, R5 to R29, R12 to R30, R9 to R31, R17 to R32, R14 to R33, R11 to R36, R10 to R37, R16 to R38, R15 to R39, R26 to R40, R27 to R41, R13 to R42, R8 to R43, R19 to R5, R18 to R6, R34 to R7, S2 to S1, S4 to S2, S6 to S3, SW3 to SW1, U5 to U14, U7 to U2, U1 to U6, U2 to U7
Connections:
- net +3.3V: now also C22.1, C15.1, C17.1, U1.16 (VDD), U10.8 (VCC), U11.1 (CPVDD), U11.20 (DVDD), U11.8 (AVDD), U12.2 (3V3), U9.2 (VCC)
- net +5V: now also C16.2, D4.1 (K), R15.1, R17.1; no longer S3.3
- net 595_CLOCK: now also U12.26 (IO4)
- net 595_DATA: now also U12.25 (IO0)
- net 595_LATCH: now also U12.24 (IO2)
- net AYMIX_L: now also R45.1
- net AYMIX_R: now also R44.1
- net AY_CLK: now also U12.14 (IO12/H_MISO)
- net Bat+: now also J2.1, Q1.2 (S), U5.5 (BAT), U9.6 (VBAT); no longer L1.2
- net ENC_A: now also U1.4 (P0)
- net ENC_B: now also U1.5 (P1)
- net ENC_OK: now also U1.6 (P2)
- net ESP_EN: now also U12.3 (EN/RST)
- net GND: now also C30.2, D5.1 (K), C14.1, C15.2, C16.1, C17.2, C24.1, C25.1, C27.2, C29.1, C31.1, J2.2, R16.2, R8.2, R9.2, U1.1 (A0), U1.2 (A1), U1.3 (A2), U1.8 (GND), U10.1 (A0), U10.2 (A1), U10.3 (A2), U10.4 (GND), U10.7 (WP), U11.10 (DEMP), U11.11 (FLT), U11.12 (SCK), U11.16 (FMT), U11.19 (DGND), U11.3 (CPGND), U11.9 (AGND), U12.1 (GND), U12.15 (GND), U12.38 (GND), U5.1 (TEMP), U5.3 (GND), U5.9 (EPAD), U8.2 (GND), U9.5 (GND); no longer C23.2, C30.1
- net SCL: now also U1.14 (SCL), U10.6 (SCL), U12.36 (IO22/SCL), U9.7 (SDA)
- net SDA: now also U1.15 (SDA), U10.5 (SDA), U12.33 (IO21/SDA), U9.8 (SCL)
- net SD_CS: now also U12.29 (IO5/V_CS)
- net SPI_CLK: now also U12.30 (IO18/V_CLK)
- net SPI_MISO: now also U12.31 (IO19/V_MISO)
- net SPI_MOSI: now also U12.37 (IO23/V_MOSI)
- net TFT_CLK: now also U12.13 (IO14/H_CLK)
- net TFT_CS: now also U12.23 (IO15/H_CS)
- net TFT_DC: now also U12.8 (IO32)
- net TFT_MOSI: now also U12.16 (IO13/H_MOSI)
- net TFT_PWM: now also U12.9 (IO33)
- net USB_SENS: now also U1.12 (P7)
- net Vin: now also D3.2 (A), Q1.1 (G), R4.1, R9.1, U5.4 (V_{CC}), U5.8 (CE)
- net Vsens: now also U12.4 (SENSOR_VP/I36)
- net at R27.2: now also U12.34 (IO3/RXD0)
- net at R26.2: now also U12.35 (IO1/TXD0)
- net at L1.1: now also S3.1, C14.2, U8.4 (EN), U8.5 (VIN)
- net at D2.1 (K): now also U5.7 (~{CHRG}); no longer D1.2 (A)
- net BT_DN renamed BTN_DN
- net BTN_DN: now also U1.7 (P3)
- net BT_UP renamed BTN_UP
- net BTN_UP: now also U1.9 (P4)
- net DAC_SOUND_L renamed DAC_BCK
- net DAC_BCK: now also U11.13 (BCK), U12.10 (IO25/DAC1)
- net DAC_SOUND_R renamed DAC_DAT
- net DAC_DAT: now also U11.14 (DIN), U12.11 (IO26/DAC2)
- new net: D4.2 (A), L1.2, U8.1 (SW)
- new net: C26.2, R22.2
- new net: C23.1, U11.4 (CAPM)
- new net: C23.2, U11.2 (CAPP)
- new net: C29.2, C31.2, U11.18 (LDOO)
- new net: C24.2, C25.2, U11.5 (VNEG)
- new net: R22.1, U11.6 (OUTL)
- new net: R23.1, U11.7 (OUTR)
- new net: D5.2 (A), R17.2
- new net: R8.1, U5.2 (PROG)
- new net: D1.1 (K), U5.6 (~{STDBY})
- new net: R15.2, R16.1, U8.3 (FB)
- new net: D1.2 (A), D2.2 (A), R4.2
- new net: C28.2, R23.2
- new net DAC_LRCK: U11.15 (LRCK), U12.12 (IO27)
- new net PCM_L: C26.1, C27.1, R45.2
- new net PCM_R: C28.1, C30.1, R44.2
- new net STPUP_VIN: D3.1 (K), Q1.3 (D), S3.2, S3.3
- no-connect marks 55 -> 58
Other:
- note added: "* In case of using external DAC: - solder all the components described in this block - do not populate R38, R39"
- note added: "* In case of using internal DAC: - do not solder components described in this block - populate R38, R39"
- note added: "*R16 value should be adjusted to limit the charging current: 2k is for ~500mA"
- note added: "Extender"
- note added: "External DAC*"
- note added: "Please note: in case of using CH340G please populate Y1, C36, C37"
- note added: "RTC & EEPROM"
- note added: "USB Charger and step-up"
- note removed: "Please make sure to use exactly the same IP5306 IC. Other ICs (like FM5324, SM5308) has some issues with sleep/wakeup modes."
- note removed: "USB Charger and step-up SoC"
- moved on the sheet: BAT+1, BAT-1, C1, C10, C11, C13, C19, C2, C20, C21, C32, C33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
