File: PCB/revD/KiCad/ESP32AY-revD.kicad_pcb (KiCad board)
At the start: 2 copper layers, 55 x 100 mm, 122 parts, among them J1 USB_C_Receptacle_USB2.0_14P, J2 Battery, J3 SD Card, J4 MiniJack, Q1 IRLML6402, Q2 BC807, SW1 BOOT, SW2 EN, U1 AMS1117-3.3, U10 PCM5102A, U11 ESP32-S3-WROOM-1, U12 TPA6130A2RTJTG4, U2 74HC595, U3 74HC595, U4 TP4056, U5 AY-3-8910, U6 DS3231MZ, U7 AY-3-8910, U8 SDB628, U9 MB85RC256V

Commit message: Some PCB and code fixes
Parts:
- U9: value MB85RC256V -> 24С32
Changed lines of the file:
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@@
 			(psa4output no)
 			(plot_black_and_white yes)
+			(plotinvisibletext no)
 			(sketchpadsonfab no)
 			(plotpadnumbers no)
@@
 		(sheetname "/")
 		(sheetfile "ESP32AY-revD.kicad_sch")
-		(attr smd exclude_from_bom dnp)
+		(attr smd)
 		(fp_line
 			(start 0.227064 0.735)
@@
 		(sheetname "/")
 		(sheetfile "ESP32AY-revD.kicad_sch")
-		(attr smd exclude_from_bom dnp)
+		(attr smd)
 		(fp_line
 			(start 2.2 -1.7)
@@
 		(sheetname "/")
 		(sheetfile "ESP32AY-revD.kicad_sch")
-		(attr smd exclude_from_bom dnp)
+		(attr smd)
 		(fp_line
 			(start 0.227064 -0.735)
@@
 			)
 		)
-		(property "Value" "MB85RC256V"
+		(property "Value" "24С32"
 			(at 0 -3.4 180)
 			(layer "B.Fab")
@@
 		(sheetname "/")
 		(sheetfile "ESP32AY-revD.kicad_sch")
-		(attr smd dnp)
+		(attr smd)
 		(fp_line
 			(start 2.2 -1.7)
