File: PCB/revD/KiCad/ESP32AY-revD.kicad_sch (KiCad schematic)
At the start: 117 parts, among them J1 USB_C_Receptacle_USB2.0_14P, J2 Battery, J3 SD Card, J4 MiniJack, Q1 IRLML6402, Q2 BC807, SW1 BOOT, SW2 EN, U1 AMS1117-3.3, U10 PCM5102A, U11 ESP32-S3-WROOM-1, U12 TPA6130A2RTJTG4, U2 74HC595, U3 74HC595, U4 TP4056, U5 AY-3-8910, U6 DS3231MZ, U7 AY-3-8910, U8 SDB628, U9 MB85RC256V

Commit message: Some PCB and code fixes
Parts:
- R17, R19, SW2: now fitted; now in the parts list
- SW1: now fitted
- U9: value MB85RC256V -> 24С32
Changed lines of the file:
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@@
 		(unit 1)
 		(exclude_from_sim no)
-		(in_bom no)
+		(in_bom yes)
 		(on_board yes)
-		(dnp yes)
+		(dnp no)
 		(fields_autoplaced yes)
 		(property "Reference" "SW2"
@@
 		(in_bom yes)
 		(on_board yes)
-		(dnp yes)
+		(dnp no)
 		(fields_autoplaced yes)
 		(property "Reference" "SW1"
@@
 		(unit 1)
 		(exclude_from_sim no)
-		(in_bom no)
+		(in_bom yes)
 		(on_board yes)
-		(dnp yes)
+		(dnp no)
 		(property "Reference" "R17"
 			(at 109.474 205.994 0)
@@
 		(unit 1)
 		(exclude_from_sim no)
-		(in_bom no)
+		(in_bom yes)
 		(on_board yes)
-		(dnp yes)
+		(dnp no)
 		(property "Reference" "R19"
 			(at 121.92 205.994 0)
@@
 			)
 		)
-		(property "Value" "MB85RC256V"
+		(property "Value" "24С32"
 			(at 185.0233 201.93 0)
 			(effects
